Commit message: Done first ever gazebo simulation launch file

File: src/bumperbot_description/urdf/bumperbot.urdf.xacro (robot description, xacro)
@@ -1,6 +1,13 @@
 <?xml version="1.0"?>
 <robot xmlns:xacro="http://www.ros.org/wiki/xacro" name="bumperbot">
+    <xacro:include filename="$(find bumperbot_description)/urdf/bumperbot_gazebo.xacro" />
     <link name="base_footprint"/>
     <link name="base_link">
+        <inertial>
+            <origin xyz="0 0 0.04" rpy="0.0 0.25 0.3" />
+            <mass value="8.2573504e-01"/>
+            <inertia ixx="2.2124416e-02" ixy="-1.2294101e-04" ixz="3.4938785e-04"
+                     iyy="2.1193702e-02" iyz="-5.0120904e-05" izz="2.0064271e-02" />
+        </inertial>
         <visual>
             <origin rpy="0 0 0" xyz="0 0 0"/>
@@ -9,4 +16,10 @@
             </geometry>
         </visual>
+        <collision>
+            <origin rpy="0 0 0" xyz="0 0 0"/>
+            <geometry>
+                <mesh filename="package://bumperbot_description/meshes/base_link.STL"/>
+            </geometry>
+        </collision>
     </link>
     <joint name="base_joint" type="fixed">
@@ -16,4 +29,11 @@
     </joint>
     <link name="wheel_right_link">
+        <inertial>
+            <origin xyz="0 -0.014 0" rpy="0 0 0" />
+            <mass value="0.0530086090966721" />
+            <inertia ixx="1.88176298336665E-05" ixy="-4.8444933029987E-10" ixz="1.88163708851143E-08"
+               iyy="3.11510738647764E-05" iyz="-6.93560663069607E-11"
+               izz="1.8801969558182E-05" />
+        </inertial>
         <visual>
             <origin rpy="1.57 0 0" xyz="0 0 0"/>
@@ -22,4 +42,10 @@
             </geometry>
         </visual>
+        <collision>
+            <origin rpy="1.57 0 0" xyz="0 -0.015 0"/>
+            <geometry>
+                <sphere radius="0.033"/>
+            </geometry>
+        </collision>
     </link>
     <joint name="wheel_right_joint" type="continuous">
@@ -30,4 +56,11 @@
     </joint>
     <link name="wheel_left_link">
+        <inertial>
+            <origin xyz="0 0.014 0" rpy="0 0 0" />
+            <mass value="0.0530086043217644" />
+            <inertia ixx="1.8792911368909E-05"  ixy="3.31256392204584E-10" ixz="-1.14082001662767E-08"
+               iyy="3.11510738759073E-05" iyz="-3.60499245082192E-10"
+               izz="1.88266886146847E-05" />
+        </inertial>
         <visual>
             <origin rpy="-1.57 0 0" xyz="0 0 0"/>
@@ -36,4 +69,10 @@
             </geometry>
         </visual>
+        <collision>
+            <origin rpy="1.57 0 0" xyz="0 0.015 0"/>
+            <geometry>
+                <sphere radius="0.033"/>
+            </geometry>
+        </collision>
     </link>
     <joint name="wheel_left_joint" type="continuous">
@@ -44,4 +83,11 @@
     </joint>
     <link name="caster_front_link">
+        <inertial>
+            <origin xyz="3.89968128948481E-07 2.40073004698083E-07 0.00219173397061506" rpy="0 0 0" />
+            <mass value="1.44379265037903E-06" />
+            <inertia ixx="7.23075276010246E-11" ixy="-6.10956883467859E-16" ixz="2.22849693525031E-15"
+               iyy="3.8713793085917E-11"  iyz="2.93909858781952E-15"
+               izz="1.00967486676306E-10" />
+        </inertial>
         <visual>
             <origin rpy="0 0 0" xyz="0 0 0"/>
@@ -50,4 +96,10 @@
             </geometry>
         </visual>
+        <collision>
+            <origin rpy="0 0 0" xyz="0 0 0"/>
+            <geometry>
+                <sphere radius="0.005"/>
+            </geometry>
+        </collision>
     </link>
     <joint name="caster_front_joint" type="fixed">
@@ -57,4 +109,11 @@
     </joint>
     <link name="caster_rear_link">
+        <inertial>
+            <origin xyz="3.8996812895542E-07 2.40073004698083E-07 0.00219173397061509" rpy="0 0 0" />
+            <mass value="1.44379265037902E-06" />
+            <inertia ixx="7.23075276010246E-11" ixy="-6.10956872363424E-16" ixz="2.22849693527207E-15"
+               iyy="3.87137930859167E-11" iyz="2.939098587861E-15"
+               izz="1.00967486676306E-10" />
+        </inertial>
         <visual>
             <origin rpy="0 0 0" xyz="0 0 0"/>
@@ -63,4 +122,10 @@
             </geometry>
         </visual>
+        <collision>
+            <origin rpy="0 0 0" xyz="0 0 0"/>
+            <geometry>
+                <sphere radius="0.005"/>
+            </geometry>
+        </collision>
     </link>
     <joint name="caster_rear_joint" type="fixed">

Commit message: controllers and bumperbot is loading and shown properly with additional timeraction module

File: src/bumperbot_description/urdf/bumperbot.urdf.xacro (robot description, xacro)
@@ -4,5 +4,5 @@
     <!--Include Gazebo Paramaters-->
     <xacro:include filename="$(find bumperbot_description)/urdf/bumperbot_gazebo.xacro" />
-    <!--ROS2 Control-->
+    <!--ROS 2 Control-->
     <xacro:include filename="$(find bumperbot_description)/urdf/bumperbot_ros2_control.xacro" />
     <link name="base_footprint"/>
@@ -17,5 +17,5 @@
             <origin rpy="0 0 0" xyz="0 0 0"/>
             <geometry>
-                <mesh filename="file:///home/ven-zenitsu/kilted_ws_ros2/src/bumperbot_description/meshes/base_link.STL"/>
+                <mesh filename="package://bumperbot_description/meshes/base_link.STL"/>
             </geometry>
         </visual>
@@ -43,5 +43,5 @@
             <origin rpy="1.57 0 0" xyz="0 0 0"/>
             <geometry>
-                <mesh filename="file:///home/ven-zenitsu/kilted_ws_ros2/src/bumperbot_description/meshes/wheel_right_link.STL"/>
+                <mesh filename="package://bumperbot_description/meshes/wheel_right_link.STL"/>
             </geometry>
         </visual>
@@ -70,5 +70,5 @@
             <origin rpy="-1.57 0 0" xyz="0 0 0"/>
             <geometry>
-                <mesh filename="file:///home/ven-zenitsu/kilted_ws_ros2/src/bumperbot_description/meshes/wheel_left_link.STL"/>
+                <mesh filename="package://bumperbot_description/meshes/wheel_left_link.STL"/>
             </geometry>
         </visual>
@@ -97,5 +97,5 @@
             <origin rpy="0 0 0" xyz="0 0 0"/>
             <geometry>
-                <mesh filename="file:///home/ven-zenitsu/kilted_ws_ros2/src/bumperbot_description/meshes/caster_front_link.STL"/>
+                <mesh filename="package://bumperbot_description/meshes/caster_front_link.STL"/>
             </geometry>
         </visual>
@@ -123,5 +123,5 @@
             <origin rpy="0 0 0" xyz="0 0 0"/>
             <geometry>
-                <mesh filename="file:///home/ven-zenitsu/kilted_ws_ros2/src/bumperbot_description/meshes/caster_rear_link.STL"/>
+                <mesh filename="package://bumperbot_description/meshes/caster_rear_link.STL"/>
             </geometry>
         </visual>

File: src/bumperbot_description/urdf/bumperbot_gazebo.xacro (robot description, xacro)
@@ -37,15 +37,14 @@
     <gazebo>
         <xacro:if value="$(arg is_ignition)">
-            <plugin filename="ign_ros2_control-system" name="ign_ros2_control::IgnitionROS2ControlPlugin">
-                <paramaters>
-                </paramaters>
+            <plugin filename="gz_ros2_control-system" name="gz_ros2_control::GazeboRos2ControlPlugin">
+                <parameters>$(find bumperbot_controller)/config/bumperbot_controllers.yaml</parameters>
             </plugin>
         </xacro:if>
         <xacro:unless value="$(arg is_ignition)">
-            <plugin filename="gz_ros2_control-system" name="gz_ros2_control::GazeboSimRos2ControlPlugin">
-                <paramaters>
-                </paramaters>
+            <plugin filename="libgz_ros2_control-system.so" name="gz_ros2_control::GazeboSimROS2ControlPlugin">
+                <parameters>$(find bumperbot_controller)/config/bumperbot_controllers.yaml</parameters>
             </plugin>
         </xacro:unless>
+        <plugin name="gazebo_ros_clock" filename="libgazebo_ros_clock.so"/>
     </gazebo>
 </robot>
